File: eagle/simpler dj midi controlle.brd (EAGLE design)
At the start: 100.3 x 39 mm, 6 parts, among them SW1 ROTARTY_ENCODER, SW2 ROTARTY_ENCODER, SW3 ROTARTY_ENCODER

Commit message: modified documentation
Parts:
- added S3: (no value), switch:320-916
Connections:
- new net N$10: S3.1, U$1.14
- net GND: now also S3.2
Changed lines of the file:
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@@
 <?xml version="1.0" encoding="utf-8"?>
 <!DOCTYPE eagle SYSTEM "eagle.dtd">
-<eagle version="9.4.0">
+<eagle version="9.2.2">
 <drawing>
 <settings>
@@
 </autorouter>
 <elements>
-<element name="S1" library="switch-omron" library_urn="urn:adsk.eagle:library:377" package="B3F-10XX" package3d_urn="urn:adsk.eagle:package:27496/1" value=""  x="39.37" y="5.08" smashed="yes">
+<element name="S1" library="switch-omron" library_urn="urn:adsk.eagle:library:377" package="B3F-10XX" package3d_urn="urn:adsk.eagle:package:27496/1" value="" x="39.37" y="5.08" smashed="yes">
 <attribute name="MF" value="" x="63.5" y="-49.53" size="1.778" layer="27" display="off"/>
 <attribute name="MPN" value="B3F-1000" x="63.5" y="-49.53" size="1.778" layer="27" display="off"/>
@@
 <attribute name="VALUE" x="11.43" y="26.67" size="0.4064" layer="27" rot="R180"/>
 </element>
-<element name="SW3" library="SparkFun-Electromechanical" package="ROTARY_ENC_PLAIN" value="ROTARTY_ENCODER"  x="86.36" y="15.24" smashed="yes" rot="R180">
+<element name="SW3" library="SparkFun-Electromechanical" package="ROTARY_ENC_PLAIN" value="ROTARTY_ENCODER" x="86.36" y="15.24" smashed="yes" rot="R180">
 <attribute name="NAME" x="86.36" y="16.51" size="0.4064" layer="25" rot="R180"/>
 <attribute name="VALUE" x="87.63" y="13.97" size="0.4064" layer="27" rot="R180"/>
@@
 <attribute name="NAME" x="64.77" y="34.29" size="1.27" layer="25"/>
 <attribute name="VALUE" x="64.77" y="36.195" size="1.27" layer="27"/>
+</element>
+<element name="S3" library="switch" library_urn="urn:adsk.eagle:library:380" package="320-916" package3d_urn="urn:adsk.eagle:package:27678/1" value="" x="-10.16" y="10.16" smashed="yes">
+<attribute name="NAME" x="-12.7" y="17.78" size="1.778" layer="25" ratio="10"/>
+<attribute name="POPULARITY" value="4" x="-10.16" y="10.16" size="1.778" layer="27" display="off"/>
+<attribute name="VALUE" x="-12.7" y="0.635" size="1.778" layer="27" ratio="10"/>
 </element>
 </elements>
@@
 <contactref element="U$1" pad="23"/>
 <contactref element="SW1" pad="SW-"/>
-<wire x1="76.2" y1="33.02" x2="93.345" y2="17.78" width="0" layer="19" extent="1-1"/>
-<wire x1="60.96" y1="27.94" x2="76.2" y2="33.02" width="0" layer="19" extent="1-1"/>
-<wire x1="47.625" y1="30.48" x2="60.96" y2="27.94" width="0" layer="19" extent="1-1"/>
-<wire x1="33.147" y1="27.94" x2="47.625" y2="30.48" width="0" layer="19" extent="1-1"/>
-<wire x1="42.4688" y1="4.0894" x2="33.147" y2="27.94" width="0" layer="19" extent="1-1"/>
-<wire x1="48.9712" y1="4.0894" x2="42.4688" y2="4.0894" width="0" layer="19" extent="1-1"/>
-<wire x1="19.685" y1="30.48" x2="33.147" y2="27.94" width="0" layer="19" extent="1-1"/>
-<wire x1="5.207" y1="27.94" x2="19.685" y2="30.48" width="0" layer="19" extent="1-1"/>
-<wire x1="14.5288" y1="4.0894" x2="5.207" y2="27.94" width="0" layer="19" extent="1-1"/>
-<wire x1="21.0312" y1="4.0894" x2="14.5288" y2="4.0894" width="0" layer="19" extent="1-1"/>
+<contactref element="S3" pad="2"/>
+<wire x1="78.867" y1="15.24" x2="93.345" y2="17.78" width="0" layer="19" extent="1-1"/>
+<wire x1="76.2" y1="30.48" x2="78.867" y2="15.24" width="0" layer="19" extent="1-1"/>
+<wire x1="60.96" y1="25.4" x2="76.2" y2="30.48" width="0" layer="19" extent="1-1"/>
+<wire x1="50.165" y1="30.48" x2="60.96" y2="25.4" width="0" layer="19" extent="1-1"/>
+<wire x1="42.6212" y1="2.8194" x2="50.165" y2="30.48" width="0" layer="19" extent="1-1"/>
+<wire x1="36.1188" y1="2.8194" x2="42.6212" y2="2.8194" width="0" layer="19" extent="1-1"/>
+<wire x1="18.4912" y1="2.8194" x2="36.1188" y2="2.8194" width="0" layer="19" extent="1-1"/>
+<wire x1="11.9888" y1="2.8194" x2="18.4912" y2="2.8194" width="0" layer="19" extent="1-1"/>
+<wire x1="-10.16" y1="10.16" x2="11.9888" y2="2.8194" width="0" layer="19" extent="1-1"/>
+<wire x1="2.667" y1="27.94" x2="-10.16" y2="10.16" width="0" layer="19" extent="1-1"/>
+<wire x1="17.145" y1="30.48" x2="2.667" y2="27.94" width="0" layer="19" extent="1-1"/>
 </signal>
 <signal name="N$11">
@@
 <wire x1="76.2" y1="17.78" x2="78.867" y2="17.78" width="0" layer="19" extent="1-1"/>
 </signal>
+<signal name="N$10">
+<contactref element="U$1" pad="14"/>
+<contactref element="S3" pad="1"/>
+<wire x1="-10.16" y1="14.1732" x2="76.2" y2="7.62" width="0" layer="19" extent="1-1"/>
+</signal>
 </signals>
