File: eagle/simpler dj midi controlle.sch (EAGLE design)
At the start: 6 parts, among them SW1 ROTARTY_ENCODER, SW2 ROTARTY_ENCODER, SW3 ROTARTY_ENCODER

Commit message: modified documentation
Parts:
- added S3: (no value), switch:320-916
Connections:
- new net N$10: S3.O, U$1.11
- net GND: now also S3.P
Changed lines of the file:
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@@
 <?xml version="1.0" encoding="utf-8"?>
 <!DOCTYPE eagle SYSTEM "eagle.dtd">
-<eagle version="9.4.0">
+<eagle version="9.2.2">
 <drawing>
 <settings>
@@
 <part name="GND4" library="supply1" library_urn="urn:adsk.eagle:library:371" deviceset="GND" device=""/>
 <part name="GND6" library="supply1" library_urn="urn:adsk.eagle:library:371" deviceset="GND" device=""/>
+<part name="S3" library="switch" library_urn="urn:adsk.eagle:library:380" deviceset="320-916" device="" package3d_urn="urn:adsk.eagle:package:27678/1"/>
+<part name="GND7" library="supply1" library_urn="urn:adsk.eagle:library:371" deviceset="GND" device=""/>
 </parts>
 <sheets>
@@
 <instance part="GND6" gate="1" x="195.58" y="124.46" smashed="yes">
 <attribute name="VALUE" x="193.04" y="121.92" size="1.778" layer="96"/>
+</instance>
+<instance part="S3" gate="1" x="142.24" y="78.74" smashed="yes">
+<attribute name="NAME" x="135.89" y="76.835" size="1.778" layer="95" rot="R90"/>
+<attribute name="VALUE" x="138.43" y="81.28" size="1.778" layer="96" rot="R90"/>
+</instance>
+<instance part="GND7" gate="1" x="144.78" y="58.42" smashed="yes">
+<attribute name="VALUE" x="142.24" y="55.88" size="1.778" layer="96"/>
 </instance>
 </instances>
@@
 <wire x1="195.58" y1="129.54" x2="193.04" y2="129.54" width="0.1524" layer="91"/>
 </segment>
+<segment>
+<pinref part="S3" gate="1" pin="P"/>
+<pinref part="GND7" gate="1" pin="GND"/>
+<wire x1="144.78" y1="73.66" x2="144.78" y2="60.96" width="0.1524" layer="91"/>
+</segment>
 </net>
 <net name="N$11" class="0">
@@
 </segment>
 </net>
+<net name="N$10" class="0">
+<segment>
+<pinref part="U$1" gate="G$1" pin="11"/>
+<pinref part="S3" gate="1" pin="O"/>
+<wire x1="127" y1="121.92" x2="142.24" y2="121.92" width="0.1524" layer="91"/>
+<wire x1="142.24" y1="121.92" x2="142.24" y2="83.82" width="0.1524" layer="91"/>
+</segment>
+</net>
